File: main/main.kicad_pcb (KiCad board)
At the start: 2 copper layers, 3.3 x 2.9 mm, 348 parts, among them J1 USB_C_Receptacle_USB2.0, J2 TC2030_SWD, SW1 SW_Push_45deg, SW10 SW_Push_45deg, SW11 SW_Push_45deg, SW12 SW_Push_45deg, SW13 SW_Push_45deg, SW14 SW_Push_45deg, SW15 SW_Push_45deg, SW16 SW_Push_45deg, SW17 SW_Push_45deg, SW18 SW_Push_45deg, SW19 SW_Push_45deg, SW2 SW_Push_45deg, SW20 SW_Push_45deg, SW21 SW_Push_45deg, SW22 SW_Push_45deg, SW23 SW_Push_45deg, SW24 SW_Push_45deg, SW25 SW_Push_45deg, SW26 SW_Push_45deg, SW27 SW_Push_45deg, SW28 SW_Push_45deg, SW29 SW_Push_45deg, SW3 SW_Push_45deg, SW30 SW_Push_45deg, SW31 SW_Push_45deg, SW32 SW_Push_45deg, SW33 SW_Push_45deg, SW34 SW_Push_45deg, SW35 SW_Push_45deg, SW36 SW_Push_45deg, SW37 SW_Push_45deg, SW38 SW_Push_45deg, SW39 SW_Push_45deg, SW4 SW_Push_45deg, SW40 SW_Push_45deg, SW41 SW_Push_45deg, SW42 SW_Push_45deg, SW43 SW_Push_45deg, SW44 SW_Push_45deg, SW45 SW_Push_45deg, SW46 SW_Push_45deg, SW47 SW_Push_45deg, SW48 SW_Push_45deg, SW49 SW_Push_45deg, SW5 SW_Push_45deg, SW50 SW_Push_45deg, SW51 SW_Push_45deg, SW52 SW_Push_45deg, SW53 SW_Push_45deg, SW54 SW_Push_45deg, SW55 SW_Push_45deg, SW56 SW_Push_45deg, SW57 SW_Push_45deg, SW58 SW_Push_45deg, SW59 SW_Push_45deg, SW6 SW_Push_45deg, SW60 SW_Push_45deg, SW61 SW_Push_45deg, SW62 SW_Push_45deg, SW63 SW_Push_45deg, SW64 SW_Push_45deg, SW65 SW_Push_45deg, SW66 SW_Push_45deg, SW67 SW_Push_45deg, SW68 SW_Push_45deg, SW69 SW_Push_45deg, SW7 SW_Push_45deg, SW70 SW_Push_45deg, SW71 SW_Push_45deg, SW72 SW_Push_45deg, SW73 SW_Push_45deg, SW74 SW_Push_45deg, SW75 SW_Push_45deg, SW76 SW_Push_45deg, SW77 SW_Push_45deg, SW78 SW_Push_45deg, SW8 SW_Push_45deg, SW9 SW_Push_45deg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

Commit message: Keyswitches placed
Parts:
- moved SW66 497.6 mm to (209.6, 78.0)
- moved SW76 494.9 mm to (231.6, 97.5)
- moved SW68 492.8 mm to (265.7, 78.0)
- moved SW56 491.9 mm to (270.6, 58.5)
- moved SW67 486.0 mm to (229.1, 78.0)
- moved SW53 474.1 mm to (199.9, 58.5)
- moved SW77 471.0 mm to (255.9, 97.5)
- moved SW65 468.7 mm to (190.1, 78.0)
- moved SW78 452.4 mm to (280.3, 97.5)
- moved SW52 437.1 mm to (180.4, 58.5)
- moved SW54 422.1 mm to (219.4, 58.5)
- moved SW51 381.3 mm to (160.9, 58.5)
- moved SW62 377.8 mm to (131.6, 78.0)
- moved SW75 372.9 mm to (207.2, 97.5)
- moved SW55 372.4 mm to (238.9, 58.5)
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
Commit message: Start placing diodes
Parts:
- C1, C10, C11, C12, C13, C14, C15, C16, C17, C18, C19, C2, C20, C22, C23, C24, C25, C26, C27, C28, C29, C3, C30, C31, C32, C33, C34, C35, C36, C37, C38, C39, C4, C40, C41, C42, C43, C44, C45, C46, C47, C48, C49, C5, C50, C51, C52, C53, C54, C55, C56, C57, C58, C59, C6, C60, C61, C62, C63, C64, C65, C66, C67, C68, C69, C7, C70, C71, C72, C73, C74, C75, C76, C77, C78, C79, C8, C80, C81, C82, C83, C84, C85, C86, C87, C88, C89, C9, C90, C91, C92, C93, C94, C95, C96, D1, D10, D100, D101, D102, D103, D104, D105, D106, D107, D108, D109, D11, D110, D111, D112, D113, D114, D115, D116, D117, D118, D119, D12, D120, D121, D122, D123, D124, D125, D126, D127, D128, D129, D13, D130, D131, D132, D133, D134, D135, D136, D137, D138, D139, D14, D140, D141, D142, D143, D144, D145, D146, D147, D148, D149, D15, D150, D151, D152, D153, D154, D155, D156, D157, D158, D159, D16, D160, D161, D162, D163, D164, D165, D166, D167, D168, D17, D18, D19, D2, D20, D21, D22, D23, D24, D25, D26, D27, D28, D29, D3, D30, D31, D32, D33, D34, D35, D36, D37, D38, D39, D4, D40, D41, D42, D43, D44, D45, D46, D47, D48, D49, D5, D50, D51, D52, D53, D54, D55, D56, D57, D58, D59, D6, D60, D61, D62, D63, D64, D65, D66, D67, D68, D69, D7, D70, D71, D72, D73, D74, D75, D76, D77, D78, D79, D8, D80, D81, D82, D83, D84, D85, D86, D87, D88, D89, D9, D90, D91, D92, D94, D95, D96, D97, D98, D99, U1, U2, U3, U4: moved to B.Cu
- SW1, SW10, SW11, SW12, SW13, SW14, SW15, SW16, SW17, SW18, SW19, SW2, SW20, SW21, SW22, SW23, SW24, SW25, SW26, SW27, SW28, SW29, SW3, SW30, SW31, SW32, SW33, SW34, SW35, SW36, SW37, SW38, SW39, SW4, SW40, SW41, SW42, SW43, SW44, SW45, SW46, SW47, SW48, SW49, SW5, SW50, SW51, SW52, SW53, SW54, SW55, SW56, SW57, SW58, SW59, SW6, SW60, SW61, SW62, SW63, SW64, SW65, SW66, SW67, SW68, SW69, SW7, SW70, SW71, SW72, SW73, SW74, SW75, SW76, SW77, SW78, SW8, SW9: footprint chonc60:Kailh_socket_MX_optional -> keyswitches:Kailh_socket_MX
- moved D30 376.2 mm to (96.9, 141.0), turned to 90 degrees
- moved D1 358.1 mm to (92.0, 102.0), turned to 90 degrees
- moved D57 348.8 mm to (104.2, 180.0), turned to 90 degrees
- moved D16 345.6 mm to (92.0, 121.5), turned to 90 degrees
- moved C45 327.7 mm to (-317.0, -51.4), turned to 180 degrees
- moved C49 319.7 mm to (-313.0, -46.4), turned to 180 degrees
- moved C46 314.8 mm to (-307.9, -42.0), turned to 180 degrees
- moved C47 310.7 mm to (-303.9, -42.0), turned to 180 degrees
- moved C51 306.3 mm to (-294.8, -29.7), turned to 180 degrees
- moved C44 305.7 mm to (-313.0, -48.9), turned to 180 degrees
- moved C50 305.7 mm to (-317.0, -48.9), turned to 180 degrees
- moved D69 305.4 mm to (94.4, 199.5), turned to 90 degrees
- moved C41 301.6 mm to (-313.0, -51.4), turned to 180 degrees
- moved C48 300.6 mm to (-298.8, -32.2), turned to 180 degrees
- moved D119 297.4 mm to (-297.3, -50.3), turned to 180 degrees
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Connections:
- net /LED_IN renamed /Row 4/LED_OUT
- net /LED_IN_1 renamed /Row 2/LED_OUT
- net /LED_IN_2 renamed /Row 3/LED_OUT
- net /LED_IN_3 renamed /Row 0/LED_IN
- net /LED_IN_4 renamed /Row 0/LED_OUT
- net /LED_IN_5 renamed /Row 1/LED_OUT
- D168 pad 2: /LED_OUT -> (no net)
- J1 pad A8: Net-(J1-PadA8) -> (no net)
- J1 pad B8: Net-(J1-PadB8) -> (no net)
- U1 pad 1: Net-(U1-Pad1) -> (no net)
- U1 pad 10: /COL0 -> /Keyswitches/COL0
- U1 pad 11: /COL1 -> /Keyswitches/COL1
- U1 pad 12: /COL2 -> /Keyswitches/COL2
- U1 pad 13: /COL3 -> /Keyswitches/COL3
- U1 pad 14: /COL4 -> /Keyswitches/COL4
- U1 pad 15: /COL5 -> /Keyswitches/COL5
- U1 pad 16: /COL6 -> /Keyswitches/COL6
- U1 pad 17: /COL7 -> /Keyswitches/COL7
- U1 pad 18: /COL8 -> /Keyswitches/COL8
- U1 pad 19: /COL9 -> /Keyswitches/COL9
- U1 pad 2: no_connect_232 -> (no net)
- U1 pad 20: /COL10 -> /Keyswitches/COL10
- U1 pad 21: /COL11 -> /Keyswitches/COL11
- U1 pad 22: /COL12 -> /Keyswitches/COL12
- U1 pad 25: /COL13 -> /Keyswitches/COL13
- U1 pad 26: /COL14 -> /Keyswitches/COL14
- U1 pad 27: no_connect_233 -> (no net)
- U1 pad 29: no_connect_234 -> (no net)
- U1 pad 3: no_connect_235 -> (no net)
- U1 pad 30: no_connect_236 -> (no net)
- U1 pad 31: no_connect_237 -> (no net)
- U1 pad 38: no_connect_238 -> (no net)
- U1 pad 4: no_connect_239 -> (no net)
- U1 pad 40: /ROW0 -> /Keyswitches/ROW0
- U1 pad 41: /ROW1 -> /Keyswitches/ROW1
- U1 pad 42: /ROW2 -> /Keyswitches/ROW2
- U1 pad 43: /ROW3 -> /Keyswitches/ROW3
- U1 pad 44: Net-(U1-Pad44) -> (no net)
- U1 pad 45: /ROW4 -> /Keyswitches/ROW4
- U1 pad 46: /ROW5 -> /Keyswitches/ROW5
- U1 pad 5: Net-(U1-Pad5) -> (no net)
- U1 pad 6: Net-(U1-Pad6) -> (no net)
Routing:
- net /Keyswitches/COL0: track 0.00 -> 108.5 mm
- net GND: track 0.00 -> 7.40 mm, vias 0 -> 2
- net Net-(D16-Pad2): track 0.00 -> 3.32 mm
- net Net-(D1-Pad2): track 0.00 -> 3.32 mm
- net Net-(D69-Pad2): track 0.00 -> 3.32 mm
- net Net-(D57-Pad2): track 0.00 -> 3.32 mm
- net Net-(D44-Pad2): track 0.00 -> 3.32 mm
- net Net-(D30-Pad2): track 0.00 -> 3.32 mm
- net +5V: track 0.00 -> 3.05 mm
- net (no net): track 0.00 -> 0.90 mm

Commit message: Place diodes
Parts:
- moved D43 486.2 mm to (360.1, 141.0), turned to 90 degrees
- moved D56 478.5 mm to (352.8, 160.5), turned to 90 degrees
- moved D14 469.8 mm to (345.5, 102.0), turned to 90 degrees
- moved D78 455.7 mm to (362.6, 199.5), turned to 90 degrees
- moved D15 455.7 mm to (365.0, 102.0)
- moved D67 448.2 mm to (311.4, 180.0), turned to 90 degrees
- moved D42 447.0 mm to (335.8, 141.0), turned to 90 degrees
- moved D55 446.7 mm to (321.1, 160.5), turned to 90 degrees
- moved D77 442.1 mm to (338.2, 199.5), turned to 90 degrees
- moved D29 441.1 mm to (355.2, 121.5), turned to 90 degrees
- moved D68 440.6 mm to (347.9, 180.0), turned to 90 degrees
- moved D13 428.2 mm to (326.0, 102.0), turned to 90 degrees
- moved D28 427.1 mm to (326.0, 121.5), turned to 90 degrees
- moved D11 408.2 mm to (287.0, 102.0), turned to 90 degrees
- moved D76 407.4 mm to (313.8, 199.5), turned to 90 degrees
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
Commit message: Place LEDs, start routing
Parts:
- removed the C36 at (-183.1, 7.36)
- removed the C51 at (-294.8, -29.7)
- removed the C65 at (-279.4, -3.82)
- removed the C66 at (-301.6, -20.5)
- removed the C79 at (-246.6, -34.7)
- removed the C80 at (-255.8, -42.0)
- removed the C81 at (-268.9, -48.9)
- removed C92, C93, C94, C95, C96: 100nF, Capacitor_SMD:C_0603_1608Metric
- removed the D108 at (-167.4, 0.94)
- removed the D123 at (-279.1, -36.1)
- removed the D137 at (-272.8, -12.5)
- removed the D138 at (-272.8, -7.74)
- removed the D151 at (-258.3, -45.6)
- removed the D152 at (-231.0, -50.3)
- removed the D153 at (-240.1, -50.3)
- removed D164, D165, D166, D167, D168: SK6812MINI-E, chonc60:LED_SK6812_MINI_E_REVERSE
- added C21: 100nF, Capacitor_SMD:C_0603_1608Metric, B.Cu at (373.0, 108.0)
- added D93: SK6812MINI-E, chonc60:LED_SK6812_MINI_E_REVERSE, B.Cu at (373.0, 105.0)
- moved C49 712.6 mm to (368.1, 147.0), turned to 0 degrees
- moved D121 700.7 mm to (368.1, 144.0), turned to 0 degrees
- moved C48 684.7 mm to (343.8, 147.0), turned to 0 degrees
- moved C62 683.8 mm to (360.8, 166.5), turned to 0 degrees
- moved D120 658.5 mm to (343.8, 144.0), turned to 0 degrees
- moved C84 649.9 mm to (370.6, 205.5), turned to 0 degrees
- moved D134 648.8 mm to (360.8, 163.5), turned to 0 degrees
- moved C47 648.3 mm to (324.2, 147.0), turned to 0 degrees
- moved C61 647.2 mm to (329.1, 166.5), turned to 0 degrees
- moved C74 642.6 mm to (355.9, 186.0), turned to 0 degrees
- moved D119 642.6 mm to (324.2, 144.0), turned to 0 degrees
- moved D133 638.6 mm to (329.1, 163.5), turned to 0 degrees
- moved C46 637.3 mm to (304.8, 147.0), turned to 0 degrees
- moved C60 635.4 mm to (309.6, 166.5), turned to 0 degrees
- moved D146 635.0 mm to (355.9, 183.0), turned to 0 degrees
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- renumbered C37 to C36, C38 to C37, C39 to C38, C40 to C39, C41 to C40, C42 to C41, C43 to C42, C44 to C43, C45 to C44, C46 to C45, C47 to C46, C48 to C47, C49 to C48, C50 to C49, C52 to C50, C53 to C51, C54 to C52, C55 to C53, C56 to C54, C57 to C55, C58 to C56, C59 to C57, C60 to C58, C61 to C59, C62 to C60, C63 to C61, C64 to C62, C67 to C63, C68 to C64, C69 to C65, C70 to C66, C71 to C67, C72 to C68, C73 to C69, C74 to C70, C75 to C71, C76 to C72, C77 to C73, C78 to C74, C82 to C75, C83 to C76, C84 to C77, C85 to C78, C86 to C79, C87 to C80, C88 to C81, C89 to C82, C90 to C83, C91 to C84, D109 to D108, D110 to D109, D111 to D110, D112 to D111, D113 to D112, D114 to D113, D115 to D114, D116 to D115, D117 to D116, D118 to D117, D119 to D118, D120 to D119, D121 to D120, D122 to D121, D124 to D122, D125 to D123, D126 to D124, D127 to D125, D128 to D126, D129 to D127, D130 to D128, D131 to D129, D132 to D130, D133 to D131, D134 to D132, D135 to D133, D136 to D134, D139 to D135, D140 to D136, D141 to D137, D142 to D138, D143 to D139, D144 to D140, D145 to D141, D146 to D142, D147 to D143, D148 to D144, D149 to D145, D150 to D146, D154 to D147, D155 to D148, D156 to D149, D157 to D150, D158 to D151, D159 to D152, D160 to D153, D161 to D154, D162 to D155, D163 to D156
Connections:
- D107 pad 2: Net-(D107-Pad2) -> /Row 1/LED_OUT
- D108 pad 2: Net-(D109-Pad2) (its old number) -> (no net)
- D109 pad 4: Net-(D109-Pad2) (its old number) -> (no net)
- D121 pad 2: Net-(D122-Pad2) -> /Row 2/LED_OUT
- D122 pad 2: Net-(D124-Pad2) (its old number) -> (no net)
- D123 pad 2: Net-(D125-Pad2) (its old number) -> (no net)
- D123 pad 4: Net-(D124-Pad2) (its old number) -> (no net)
- D124 pad 4: Net-(D125-Pad2) (its old number) -> (no net)
- D134 pad 2: Net-(D136-Pad2) -> /Row 3/LED_OUT
- D136 pad 2: Net-(D140-Pad2) (its old number) -> (no net)
- D137 pad 2: Net-(D141-Pad2) (its old number) -> (no net)
- D137 pad 4: Net-(D140-Pad2) (its old number) -> (no net)
- D138 pad 2: Net-(D142-Pad2) (its old number) -> (no net)
- D138 pad 4: Net-(D141-Pad2) (its old number) -> (no net)
- D139 pad 4: Net-(D142-Pad2) (its old number) -> (no net)
- D146 pad 2: Net-(D150-Pad2) -> /Row 4/LED_OUT
- D150 pad 2: Net-(D157-Pad2) -> (no net)
- D151 pad 2: Net-(D158-Pad2) -> (no net)
- D151 pad 4: Net-(D157-Pad2) -> (no net)
- D152 pad 2: Net-(D159-Pad2) -> (no net)
- D152 pad 4: Net-(D158-Pad2) -> (no net)
- D153 pad 4: Net-(D159-Pad2) -> (no net)
- D156 pad 2: Net-(D163-Pad2) -> (no net)
- D92 pad 2: /Row 0/LED_OUT -> (no net)
- D94 pad 4: /Row 0/LED_OUT -> (no net)
Routing:
- net Net-(D91-Pad2): track 0.00 -> 14.7 mm
- net Net-(D90-Pad2): track 0.00 -> 14.7 mm
- net Net-(D89-Pad2): track 0.00 -> 14.7 mm
- net Net-(D88-Pad2): track 0.00 -> 14.7 mm
- net Net-(D87-Pad2): track 0.00 -> 14.7 mm
- net Net-(D86-Pad2): track 0.00 -> 14.7 mm
- net Net-(D85-Pad2): track 0.00 -> 14.7 mm
- net Net-(D84-Pad2): track 0.00 -> 14.7 mm
- net Net-(D83-Pad2): track 0.00 -> 14.7 mm
- net Net-(D82-Pad2): track 0.00 -> 14.7 mm
- net Net-(D81-Pad2): track 0.00 -> 14.7 mm
- net (no net): track 0.90 -> 15.6 mm
- net Net-(D80-Pad2): track 0.00 -> 14.7 mm
- net Net-(D79-Pad2): track 0.00 -> 14.7 mm
- net Net-(D3-Pad2): track 0.00 -> 3.32 mm
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
Commit message: Make LEDs make more sense, with automation!
Parts:
- moved C75 268.1 mm to (370.6, 205.5), turned to 180 degrees
- moved C84 268.1 mm to (102.4, 205.5), turned to 180 degrees
- moved D147 268.1 mm to (370.6, 202.5), turned to 180 degrees
- moved D156 268.1 mm to (102.4, 202.5), turned to 180 degrees
- moved C22 263.2 mm to (363.2, 127.5), turned to 180 degrees
- moved C35 263.2 mm to (100.0, 127.5), turned to 180 degrees
- moved D107 263.2 mm to (100.0, 124.5), turned to 180 degrees
- moved D94 263.2 mm to (363.2, 124.5), turned to 180 degrees
- moved C50 253.5 mm to (360.8, 166.5), turned to 180 degrees
- moved C62 253.5 mm to (107.3, 166.5), turned to 180 degrees
- moved D122 253.5 mm to (360.8, 163.5), turned to 180 degrees
- moved D134 253.5 mm to (107.3, 163.5), turned to 180 degrees
- moved C76 219.4 mm to (346.2, 205.5), turned to 180 degrees
- moved C83 219.4 mm to (126.8, 205.5), turned to 180 degrees
- moved D148 219.4 mm to (346.2, 202.5), turned to 180 degrees
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Connections:
- net Net-(J1-PadA6) renamed /C_D+
- net Net-(J1-PadA7) renamed /C_D-
- D122 pad 2: (no net) -> Net-(D122-Pad2)
- D123 pad 2: (no net) -> Net-(D123-Pad2)
- D123 pad 4: (no net) -> Net-(D122-Pad2)
- D124 pad 4: (no net) -> Net-(D123-Pad2)
- D136 pad 2: (no net) -> Net-(D136-Pad2)
- D137 pad 2: (no net) -> Net-(D137-Pad2)
- D137 pad 4: (no net) -> Net-(D136-Pad2)
- D138 pad 2: (no net) -> Net-(D138-Pad2)
- D138 pad 4: (no net) -> Net-(D137-Pad2)
- D139 pad 4: (no net) -> Net-(D138-Pad2)
- D150 pad 2: (no net) -> Net-(D150-Pad2)
- D151 pad 2: (no net) -> Net-(D151-Pad2)
- D151 pad 4: (no net) -> Net-(D150-Pad2)
- D152 pad 2: (no net) -> Net-(D152-Pad2)
- D152 pad 4: (no net) -> Net-(D151-Pad2)
- D153 pad 4: (no net) -> Net-(D152-Pad2)
- D94 pad 4: (no net) -> /Row 0/LED_OUT
Routing:
- net /Keyswitches/ROW0: track 0.00 -> 308.7 mm
- net /Keyswitches/COL1: track 0.00 -> 147.6 mm, vias 0 -> 7
- net GND: track 7.40 -> 77.1 mm, vias 2 -> 5
- net /Keyswitches/COL3: track 0.00 -> 54.0 mm, vias 0 -> 2
- net /Keyswitches/COL2: track 0.00 -> 36.2 mm, vias 0 -> 2
- net /Keyswitches/COL0: track 108.5 -> 141.1 mm, vias 0 -> 2
- net +3V3: track 0.00 -> 25.0 mm, vias 0 -> 1
- net /MCU_DOUT: track 0.00 -> 23.8 mm, vias 0 -> 2
- net +5V: track 3.05 -> 24.5 mm, vias 0 -> 2
- net /C_D-: track 0.00 -> 14.9 mm, vias 0 -> 2
- net /SWDIO: track 0.00 -> 14.1 mm, vias 0 -> 1
- net /SWCLK: track 0.00 -> 14.0 mm, vias 0 -> 1
- net /C_D+: track 0.00 -> 13.3 mm, vias 0 -> 1
- net Net-(J1-PadB5): track 0.00 -> 13.1 mm
- net /SWO: track 0.00 -> 12.3 mm, vias 0 -> 1
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
Commit message: Update to new keyboard layout
Parts:
- removed C63, C64, C65, C66, C67, C68, C69, C70, C71, C72, C73, C74: 100nF, Capacitor_SMD:C_0603_1608Metric
- removed the D135 at (112.2, 183.0)
- removed the D136 at (143.9, 183.0)
- removed the D137 at (163.4, 183.0)
- removed the D138 at (182.9, 183.0)
- removed the D139 at (202.4, 183.0)
- removed the D140 at (221.9, 183.0)
- removed the D141 at (241.4, 183.0)
- removed the D142 at (260.9, 183.0)
- removed the D143 at (280.4, 183.0)
- removed the D144 at (299.9, 183.0)
- removed the D145 at (319.4, 183.0)
- removed the D146 at (355.9, 183.0)
- added C116: 100nF, Capacitor_SMD:C_0603_1608Metric, B.Cu at (112.2, 186.0)
- added C117: 100nF, Capacitor_SMD:C_0603_1608Metric, B.Cu at (143.9, 186.0)
- added C118: 100nF, Capacitor_SMD:C_0603_1608Metric, B.Cu at (163.4, 186.0)
- added C119: 100nF, Capacitor_SMD:C_0603_1608Metric, B.Cu at (182.9, 186.0)
- added C120: 100nF, Capacitor_SMD:C_0603_1608Metric, B.Cu at (202.4, 186.0)
- added C121: 100nF, Capacitor_SMD:C_0603_1608Metric, B.Cu at (221.9, 186.0)
- added C122: 100nF, Capacitor_SMD:C_0603_1608Metric, B.Cu at (241.4, 186.0)
- added C123: 100nF, Capacitor_SMD:C_0603_1608Metric, B.Cu at (260.9, 186.0)
- added C124: 100nF, Capacitor_SMD:C_0603_1608Metric, B.Cu at (280.4, 186.0)
- added C125: 100nF, Capacitor_SMD:C_0603_1608Metric, B.Cu at (299.9, 186.0)
- added C126: 100nF, Capacitor_SMD:C_0603_1608Metric, B.Cu at (319.4, 186.0)
- added C127: 100nF, Capacitor_SMD:C_0603_1608Metric, B.Cu at (346.2, 186.0)
- added C128: 100nF, Capacitor_SMD:C_0603_1608Metric, B.Cu at (373.0, 186.0)
- added C180: 100nF, Capacitor_SMD:C_0603_1608Metric, B.Cu at (373.0, 205.5)
- added D116: SK6812MINI-E, chonc60:LED_SK6812_MINI_E_REVERSE, B.Cu at (112.2, 183.0)
- added D117: SK6812MINI-E, chonc60:LED_SK6812_MINI_E_REVERSE, B.Cu at (143.9, 183.0)
- added D118: SK6812MINI-E, chonc60:LED_SK6812_MINI_E_REVERSE, B.Cu at (163.4, 183.0)
- added D119: SK6812MINI-E, chonc60:LED_SK6812_MINI_E_REVERSE, B.Cu at (182.9, 183.0)
- added D120: SK6812MINI-E, chonc60:LED_SK6812_MINI_E_REVERSE, B.Cu at (202.4, 183.0)
- added D121: SK6812MINI-E, chonc60:LED_SK6812_MINI_E_REVERSE, B.Cu at (221.9, 183.0)
- added D122: SK6812MINI-E, chonc60:LED_SK6812_MINI_E_REVERSE, B.Cu at (241.4, 183.0)
- added D123: SK6812MINI-E, chonc60:LED_SK6812_MINI_E_REVERSE, B.Cu at (260.9, 183.0)
- added D124: SK6812MINI-E, chonc60:LED_SK6812_MINI_E_REVERSE, B.Cu at (280.4, 183.0)
- added D125: SK6812MINI-E, chonc60:LED_SK6812_MINI_E_REVERSE, B.Cu at (299.9, 183.0)
- added D126: SK6812MINI-E, chonc60:LED_SK6812_MINI_E_REVERSE, B.Cu at (319.4, 183.0)
- added D127: SK6812MINI-E, chonc60:LED_SK6812_MINI_E_REVERSE, B.Cu at (346.2, 183.0)
- added D128: SK6812MINI-E, chonc60:LED_SK6812_MINI_E_REVERSE, B.Cu at (373.0, 183.0)
- added D180: SK6812MINI-E, chonc60:LED_SK6812_MINI_E_REVERSE, B.Cu at (373.0, 202.5)
- added D69: D_Small, Diode_SMD:D_SOD-123F, B.Cu at (365.0, 180.0)
- added D80: D_Small, Diode_SMD:D_SOD-123F, B.Cu at (365.0, 199.5)
- added REF**: Stabilizer_MX_2u, keyswitches:Stabilizer_MX_2u, F.Cu at (112.2, 178.0)
- added REF**: Stabilizer_MX_2u, keyswitches:Stabilizer_MX_2u, F.Cu at (258.4, 197.5)
- added REF**: Stabilizer_MX_2u, keyswitches:Stabilizer_MX_2u, F.Cu at (209.7, 197.5)
- added REF**: Stabilizer_MX_2u, keyswitches:Stabilizer_MX_2u, F.Cu at (363.2, 119.5)
- added REF**: Stabilizer_MX_2u, keyswitches:Stabilizer_MX_2u, F.Cu at (360.8, 158.5)
- added SW69: SW_Push_45deg, keyswitches:Kailh_socket_MX, F.Cu at (373.0, 178.0)
- added SW80: SW_Push_45deg, keyswitches:Kailh_socket_MX, F.Cu at (373.0, 197.5)
- moved C170 17.1 mm to (353.5, 205.5)
- moved D170 17.1 mm to (353.5, 202.5)
- moved D79 17.1 mm to (345.5, 199.5)
- moved SW79 17.1 mm to (353.5, 197.5)
- moved C171 12.2 mm to (334.0, 205.5)
- moved D171 12.2 mm to (334.0, 202.5)
- moved D78 12.2 mm to (326.0, 199.5)
- moved SW78 12.2 mm to (334.0, 197.5)
- moved D68 9.75 mm to (338.2, 180.0)
- moved SW68 9.75 mm to (346.2, 178.0)
- moved C172 7.31 mm to (314.5, 205.5)
- moved D172 7.31 mm to (314.5, 202.5)
- moved D77 7.31 mm to (306.5, 199.5)
- moved SW77 7.31 mm to (314.5, 197.5)
- moved C173 2.44 mm to (295.0, 205.5)
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- renumbered C7 to C101, C8 to C102, C9 to C103, C10 to C104, C11 to C105, C12 to C106, C13 to C107, C14 to C108, C15 to C109, C16 to C110, C17 to C111, C18 to C112, C19 to C113, C20 to C114, C21 to C115, C22 to C129, C23 to C130, C24 to C131, C25 to C132, C26 to C133, C27 to C134, C28 to C135, C29 to C136, C30 to C137, C31 to C138, C32 to C139, C33 to C140, C34 to C141, C35 to C142, C36 to C143, C37 to C144, C38 to C145, C39 to C146, C40 to C147, C41 to C148, C42 to C149, C43 to C150, C44 to C151, C45 to C152, C46 to C153, C47 to C154, C48 to C155, C49 to C156, C50 to C157, C51 to C158, C52 to C159, C53 to C160, C54 to C161, C55 to C162, C56 to C163, C57 to C164, C58 to C165, C59 to C166, C60 to C167, C61 to C168, C62 to C169, C75 to C170, C76 to C171, C77 to C172, C78 to C173, C79 to C174, C80 to C175, C81 to C176, C82 to C177, C83 to C178, C84 to C179, D79 to D101, D80 to D102, D81 to D103, D82 to D104, D83 to D105, D84 to D106, D85 to D107, D86 to D108, D87 to D109, D88 to D110, D89 to D111, D90 to D112, D91 to D113, D92 to D114, D93 to D115, D94 to D129, D95 to D130, D96 to D131, D97 to D132, D98 to D133, D99 to D134, D100 to D135, D101 to D136, D102 to D137, D103 to D138, D104 to D139, D105 to D140, D106 to D141, D107 to D142, D108 to D143, D109 to D144, D110 to D145, D111 to D146, D112 to D147, D113 to D148, D114 to D149, D115 to D150, D116 to D151, D117 to D152, D118 to D153, D119 to D154, D120 to D155, D121 to D156, D122 to D157, D123 to D158, D124 to D159, D125 to D160, D126 to D161, D127 to D162, D128 to D163, D129 to D164, D130 to D165, D131 to D166, D132 to D167, D133 to D168, D134 to D169, D147 to D170, D148 to D171, D149 to D172, D150 to D173, D151 to D174, D152 to D175, D153 to D176, D154 to D177, D155 to D178, D156 to D179, D69 to D70, D70 to D71, D71 to D72, D72 to D73, D73 to D74, D74 to D75, D75 to D76, D76 to D77, D77 to D78, D78 to D79, SW69 to SW70, SW70 to SW71, SW71 to SW72, SW72 to SW73, SW73 to SW74, SW74 to SW75, SW75 to SW76, SW76 to SW77, SW77 to SW78, SW78 to SW79
Connections:
- D114 pad 2: (no net) -> Net-(D114-Pad2)
- D115 pad 4: (no net) -> Net-(D114-Pad2)
- D143 pad 2: (no net) -> Net-(D143-Pad2)
- D144 pad 4: (no net) -> Net-(D143-Pad2)
- D179 pad 2: (no net) -> Net-(D179-Pad2)
- D76 pad 1: /Keyswitches/COL11 -> /Keyswitches/COL10
- D77 pad 1: /Keyswitches/COL12 -> /Keyswitches/COL11
- D78 pad 1: /Keyswitches/COL13 -> /Keyswitches/COL12
- D79 pad 1: /Keyswitches/COL14 -> /Keyswitches/COL13
- J1 pad A8: (no net) -> unconnected-(J1-PadA8)
- J1 pad B8: (no net) -> unconnected-(J1-PadB8)
- SW76 pad 1: /Keyswitches/ROW5 -> unconnected-(SW76-Pad1)
- U1 pad 1: (no net) -> unconnected-(U1-Pad1)
- U1 pad 2: (no net) -> unconnected-(U1-Pad2)
- U1 pad 27: (no net) -> unconnected-(U1-Pad27)
- U1 pad 29: (no net) -> unconnected-(U1-Pad29)
- U1 pad 3: (no net) -> unconnected-(U1-Pad3)
- U1 pad 30: (no net) -> unconnected-(U1-Pad30)
- U1 pad 31: (no net) -> unconnected-(U1-Pad31)
- U1 pad 38: (no net) -> unconnected-(U1-Pad38)
- U1 pad 4: (no net) -> unconnected-(U1-Pad4)
- U1 pad 44: (no net) -> unconnected-(U1-Pad44)
- U1 pad 5: (no net) -> Net-(U1-Pad5)
- U1 pad 6: (no net) -> Net-(U1-Pad6)
- U2 pad 1: (no net) -> unconnected-(U2-Pad1)
- U4 pad 4: (no net) -> unconnected-(U4-Pad4)
Routing:
- net Net-(D114-Pad2): track 0.00 -> 14.7 mm
- net (no net): track 15.6 -> 0.90 mm
- net +3V3: track 25.0 -> 35.8 mm
- net GND: track 77.1 -> 85.8 mm
- net /Keyswitches/COL0: track 141.1 -> 146.5 mm
- net Net-(D80-Pad2): track 0.00 -> 3.32 mm
- net Net-(D69-Pad2): track 0.00 -> 3.32 mm
Other:
- board size 3.3 x 2.9 mm -> 295 x 130 mm

Commit message: Move around parts, some matrix routing
Parts:
- R1, R2: moved to B.Cu
- moved U3 275.4 mm to (382.5, 168.4), turned to -90 degrees
- moved J1 265.3 mm to (381.7, 158.8), turned to 90 degrees
- moved R1 259.0 mm to (382.9, 161.1), turned to 0 degrees
- moved R2 256.1 mm to (382.9, 156.4), turned to 0 degrees
- moved U2 195.8 mm to (241.5, 219.4)
- moved C5 186.3 mm to (280.7, 195.2)
- moved U4 185.1 mm to (275.8, 195.8)
- moved C6 184.8 mm to (271.9, 195.4)
- moved C4 174.8 mm to (230.6, 204.7), turned to 0 degrees
- moved C3 174.0 mm to (240.0, 201.8)
- moved U1 166.8 mm to (233.6, 198.4)
- moved C2 158.4 mm to (237.2, 191.8), turned to 180 degrees
- moved C1 158.3 mm to (225.5, 197.3), turned to -90 degrees
- moved J2 142.8 mm to (189.6, 198.2)
Routing:
- net /Keyswitches/ROW1: track 0.00 -> 326.9 mm
- net /Keyswitches/ROW2: track 0.00 -> 325.8 mm
- net /Keyswitches/ROW3: track 0.00 -> 324.7 mm
- net /USB_D+: track 3.91 -> 186.3 mm
- net /USB_D-: track 3.91 -> 185.5 mm
- net /Keyswitches/COL2: track 36.2 -> 121.2 mm, vias 2 -> 6
- net /Keyswitches/COL3: track 54.0 -> 1.30 mm, vias 2 -> 0
- net /Keyswitches/COL0: track 146.5 -> 113.9 mm, vias 2 -> 0
- net GND: track 85.8 -> 56.8 mm, vias 5 -> 4
- net +5V: track 24.5 -> 53.5 mm, vias 2 -> 1
- net /MCU_DOUT: track 23.8 -> 0.00 mm, vias 2 -> 0
- net /Keyswitches/COL1: track 147.6 -> 123.9 mm, vias 7 -> 6
- net +3V3: track 35.8 -> 12.7 mm, vias 1 -> 0
- net /SWDIO: track 14.1 -> 0.00 mm, vias 1 -> 0
- net /SWCLK: track 14.0 -> 0.00 mm, vias 1 -> 0
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Other:
- board size 295 x 130 mm -> 297 x 121.5 mm

Commit message: Switch to STM32L063 because I can actually buy those
Parts:
- added C2: 1µF, Capacitor_SMD:C_0603_1608Metric, B.Cu at (223.8, 197.3)
- added C5: 10µF, Capacitor_SMD:C_0603_1608Metric, B.Cu at (230.6, 206.4)
- added TP1: BOOT0, TestPoint:TestPoint_Pad_D1.0mm, F.Cu at (293.8, 220.7)
- added TP2: ~RESET, TestPoint:TestPoint_Pad_D1.0mm, F.Cu at (289.7, 217.9)
- added TP3: GND, TestPoint:TestPoint_Pad_1.0x1.0mm, F.Cu at (283.2, 221.4)
- added TP4: 5V, TestPoint:TestPoint_Pad_D1.0mm, F.Cu at (289.7, 221.0)
- added TP5: 3V3, TestPoint:TestPoint_Pad_D1.0mm, F.Cu at (292.8, 217.9)
- U1: value STM32F303CBTx -> STM32L063C8Tx
- moved C3 10.4 mm to (237.1, 191.8), turned to 180 degrees
- moved C6 10.4 mm to (240.1, 201.8), turned to 90 degrees
- moved R2 10.4 mm to (372.6, 155.0), turned to 180 degrees
- moved C7 1.36 mm to (279.4, 195.6)
- moved C8 0.54 mm to (272.4, 195.6)
- renumbered C2 to C6, C5 to C7, C6 to C8
Connections:
- J2 pad 1: +3V3 -> GND
- J2 pad 2: /SWDIO -> unconnected-(J2-Pad2)
- J2 pad 3: /~RESET -> /SWCLK
- J2 pad 4: /SWCLK -> /~RESET
- J2 pad 5: GND -> +3V3
- J2 pad 6: /SWO -> /SWDIO
- SW76 pad 1: unconnected-(SW76-Pad1) -> /Keyswitches/ROW5
- U1 pad 39: /SWO -> unconnected-(U1-Pad39)
- U1 pad 44: unconnected-(U1-Pad44) -> Net-(TP1-Pad1)
- U1 pad 5: Net-(U1-Pad5) -> unconnected-(U1-Pad5)
- U1 pad 6: Net-(U1-Pad6) -> unconnected-(U1-Pad6)
Routing:
- net +5V: track 53.5 -> 208.7 mm
- net +3V3: track 12.7 -> 57.1 mm
- net GND: track 56.8 -> 74.8 mm
- net Net-(J1-PadB5): track 4.37 -> 6.71 mm
- net (no net): track 0.90 -> 0.00 mm
