File: main/led_row_13.kicad_sch (KiCad schematic)
At the start: 30 parts

Commit message: Start placing components
Parts:
- C52: renamed from C301; footprint (none) -> Capacitor_SMD:C_0603_1608Metric
- C53: renamed from C302; footprint (none) -> Capacitor_SMD:C_0603_1608Metric
- C54: renamed from C303; footprint (none) -> Capacitor_SMD:C_0603_1608Metric
- C55: renamed from C304; footprint (none) -> Capacitor_SMD:C_0603_1608Metric
- C56: renamed from C305; footprint (none) -> Capacitor_SMD:C_0603_1608Metric
- C57: renamed from C306; footprint (none) -> Capacitor_SMD:C_0603_1608Metric
- C58: renamed from C307; footprint (none) -> Capacitor_SMD:C_0603_1608Metric
- C59: renamed from C308; footprint (none) -> Capacitor_SMD:C_0603_1608Metric
- C60: renamed from C309; footprint (none) -> Capacitor_SMD:C_0603_1608Metric
- C61: renamed from C310; footprint (none) -> Capacitor_SMD:C_0603_1608Metric
- C62: renamed from C311; footprint (none) -> Capacitor_SMD:C_0603_1608Metric
- C63: renamed from C312; footprint (none) -> Capacitor_SMD:C_0603_1608Metric
- C64: renamed from C313; footprint (none) -> Capacitor_SMD:C_0603_1608Metric
- C65: renamed from C314; footprint (none) -> Capacitor_SMD:C_0603_1608Metric
- C66: renamed from C?; footprint (none) -> Capacitor_SMD:C_0603_1608Metric
- D124: renamed from D301; footprint bigbutton:LED_SK6812_MINI_E_REVERSE -> chonc60:LED_SK6812_MINI_E_REVERSE
- D125: renamed from D302; footprint bigbutton:LED_SK6812_MINI_E_REVERSE -> chonc60:LED_SK6812_MINI_E_REVERSE
- D126: renamed from D303; footprint bigbutton:LED_SK6812_MINI_E_REVERSE -> chonc60:LED_SK6812_MINI_E_REVERSE
- D127: renamed from D304; footprint bigbutton:LED_SK6812_MINI_E_REVERSE -> chonc60:LED_SK6812_MINI_E_REVERSE
- D128: renamed from D305; footprint bigbutton:LED_SK6812_MINI_E_REVERSE -> chonc60:LED_SK6812_MINI_E_REVERSE
- D129: renamed from D306; footprint bigbutton:LED_SK6812_MINI_E_REVERSE -> chonc60:LED_SK6812_MINI_E_REVERSE
- D130: renamed from D307; footprint bigbutton:LED_SK6812_MINI_E_REVERSE -> chonc60:LED_SK6812_MINI_E_REVERSE
- D131: renamed from D308; footprint bigbutton:LED_SK6812_MINI_E_REVERSE -> chonc60:LED_SK6812_MINI_E_REVERSE
- D132: renamed from D309; footprint bigbutton:LED_SK6812_MINI_E_REVERSE -> chonc60:LED_SK6812_MINI_E_REVERSE
- D133: renamed from D310; footprint bigbutton:LED_SK6812_MINI_E_REVERSE -> chonc60:LED_SK6812_MINI_E_REVERSE
- D134: renamed from D311; footprint bigbutton:LED_SK6812_MINI_E_REVERSE -> chonc60:LED_SK6812_MINI_E_REVERSE
- D135: renamed from D312; footprint bigbutton:LED_SK6812_MINI_E_REVERSE -> chonc60:LED_SK6812_MINI_E_REVERSE
- D136: renamed from D313; footprint bigbutton:LED_SK6812_MINI_E_REVERSE -> chonc60:LED_SK6812_MINI_E_REVERSE
- D137: renamed from D314; footprint bigbutton:LED_SK6812_MINI_E_REVERSE -> chonc60:LED_SK6812_MINI_E_REVERSE
- D138: renamed from D?; footprint bigbutton:LED_SK6812_MINI_E_REVERSE -> chonc60:LED_SK6812_MINI_E_REVERSE

Commit message: Place diodes
Parts:
- removed C65, C66: 100nF, Capacitor_SMD:C_0603_1608Metric, symbol Device:C_Small
- removed D137, D138: SK6812MINI-E, chonc60:LED_SK6812_MINI_E_REVERSE, symbol chonc60:SK6812MINI-E
Connections:
- net LED_OUT: now also D136.2 (DOUT)

Commit message: Place LEDs, start routing
Parts:
- renumbered C52 to C50, C53 to C51, C54 to C52, C55 to C53, C56 to C54, C57 to C55, C58 to C56, C59 to C57, C60 to C58, C61 to C59, C62 to C60, C63 to C61, C64 to C62, D124 to D122, D125 to D123, D126 to D124, D127 to D125, D128 to D126, D129 to D127, D130 to D128, D131 to D129, D132 to D130, D133 to D131, D134 to D132, D135 to D133, D136 to D134

Commit message: Update to new keyboard layout
Parts:
- renumbered C50 to C116, C51 to C117, C52 to C118, C53 to C119, C54 to C120, C55 to C121, C56 to C122, C57 to C123, C58 to C124, C59 to C125, C60 to C126, C61 to C127, C62 to C128, D122 to D116, D123 to D117, D124 to D118, D125 to D119, D126 to D120, D127 to D121, D128 to D122, D129 to D123, D130 to D124, D131 to D125, D132 to D126, D133 to D127, D134 to D128

Commit message: Switch to STM32L063 because I can actually buy those
Parts:
- renumbered C116 to C157, C117 to C158, C118 to C159, C119 to C160, C120 to C161, C121 to C162, C122 to C163, C123 to C164, C124 to C165, C125 to C166, C126 to C167, C127 to C168, C128 to C169, D116 to D157, D117 to D158, D118 to D159, D119 to D160, D120 to D161, D121 to D162, D122 to D163, D123 to D164, D124 to D165, D125 to D166, D126 to D167, D127 to D168, D128 to D169

Commit message: Start appeasing the DRC
Parts:
- renumbered C157 to C116, C158 to C117, C159 to C118, C160 to C119, C161 to C120, C162 to C121, C163 to C122, C164 to C123, C165 to C124, C166 to C125, C167 to C126, C168 to C127, C169 to C128, D157 to D116, D158 to D117, D159 to D118, D160 to D119, D161 to D120, D162 to D121, D163 to D122, D164 to D123, D165 to D124, D166 to D125, D167 to D126, D168 to D127, D169 to D128

Commit message: Convert to kicad 6.0
Parts:
- renumbered C116 to C157, C117 to C158, C118 to C159, C119 to C160, C120 to C161, C121 to C162, C122 to C163, C123 to C164, C124 to C165, C125 to C166, C126 to C167, C127 to C168, C128 to C169, D116 to D157, D117 to D158, D118 to D159, D119 to D160, D120 to D161, D121 to D162, D122 to D163, D123 to D164, D124 to D165, D125 to D166, D126 to D167, D127 to D168, D128 to D169
