File: main/led_row_13.kicad_sch (KiCad schematic)
At the start: 26 parts

Commit message: Switch to nRF58420 module and battery power
Parts:
- renumbered C157 to C46, C158 to C47, C159 to C48, C160 to C49, C161 to C50, C162 to C51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
