File: main/led_row_14.kicad_sch (KiCad schematic)
At the start: 30 parts

Commit message: Start placing components
Parts:
- C37: renamed from C82; footprint (none) -> Capacitor_SMD:C_0603_1608Metric
- C38: renamed from C83; footprint (none) -> Capacitor_SMD:C_0603_1608Metric
- C39: renamed from C84; footprint (none) -> Capacitor_SMD:C_0603_1608Metric
- C40: renamed from C85; footprint (none) -> Capacitor_SMD:C_0603_1608Metric
- C41: renamed from C86; footprint (none) -> Capacitor_SMD:C_0603_1608Metric
- C42: renamed from C87; footprint (none) -> Capacitor_SMD:C_0603_1608Metric
- C43: renamed from C88; footprint (none) -> Capacitor_SMD:C_0603_1608Metric
- C44: renamed from C89; footprint (none) -> Capacitor_SMD:C_0603_1608Metric
- C45: renamed from C90; footprint (none) -> Capacitor_SMD:C_0603_1608Metric
- C46: renamed from C91; footprint (none) -> Capacitor_SMD:C_0603_1608Metric
- C47: renamed from C92; footprint (none) -> Capacitor_SMD:C_0603_1608Metric
- C48: renamed from C93; footprint (none) -> Capacitor_SMD:C_0603_1608Metric
- C49: renamed from C94; footprint (none) -> Capacitor_SMD:C_0603_1608Metric
- C50: renamed from C95; footprint (none) -> Capacitor_SMD:C_0603_1608Metric
- C51: renamed from C96; footprint (none) -> Capacitor_SMD:C_0603_1608Metric
- D109: renamed from D154; footprint bigbutton:LED_SK6812_MINI_E_REVERSE -> chonc60:LED_SK6812_MINI_E_REVERSE
- D110: renamed from D155; footprint bigbutton:LED_SK6812_MINI_E_REVERSE -> chonc60:LED_SK6812_MINI_E_REVERSE
- D111: renamed from D156; footprint bigbutton:LED_SK6812_MINI_E_REVERSE -> chonc60:LED_SK6812_MINI_E_REVERSE
- D112: renamed from D157; footprint bigbutton:LED_SK6812_MINI_E_REVERSE -> chonc60:LED_SK6812_MINI_E_REVERSE
- D113: renamed from D158; footprint bigbutton:LED_SK6812_MINI_E_REVERSE -> chonc60:LED_SK6812_MINI_E_REVERSE
- D114: renamed from D159; footprint bigbutton:LED_SK6812_MINI_E_REVERSE -> chonc60:LED_SK6812_MINI_E_REVERSE
- D115: renamed from D160; footprint bigbutton:LED_SK6812_MINI_E_REVERSE -> chonc60:LED_SK6812_MINI_E_REVERSE
- D116: renamed from D161; footprint bigbutton:LED_SK6812_MINI_E_REVERSE -> chonc60:LED_SK6812_MINI_E_REVERSE
- D117: renamed from D162; footprint bigbutton:LED_SK6812_MINI_E_REVERSE -> chonc60:LED_SK6812_MINI_E_REVERSE
- D118: renamed from D163; footprint bigbutton:LED_SK6812_MINI_E_REVERSE -> chonc60:LED_SK6812_MINI_E_REVERSE
- D119: renamed from D164; footprint bigbutton:LED_SK6812_MINI_E_REVERSE -> chonc60:LED_SK6812_MINI_E_REVERSE
- D120: renamed from D165; footprint bigbutton:LED_SK6812_MINI_E_REVERSE -> chonc60:LED_SK6812_MINI_E_REVERSE
- D121: renamed from D166; footprint bigbutton:LED_SK6812_MINI_E_REVERSE -> chonc60:LED_SK6812_MINI_E_REVERSE
- D122: renamed from D167; footprint bigbutton:LED_SK6812_MINI_E_REVERSE -> chonc60:LED_SK6812_MINI_E_REVERSE
- D123: renamed from D168; footprint bigbutton:LED_SK6812_MINI_E_REVERSE -> chonc60:LED_SK6812_MINI_E_REVERSE

Commit message: Place diodes
Parts:
- removed C51: 100nF, Capacitor_SMD:C_0603_1608Metric, symbol Device:C_Small
- removed D123: SK6812MINI-E, chonc60:LED_SK6812_MINI_E_REVERSE, symbol chonc60:SK6812MINI-E
- renumbered C37 to C22, C38 to C23, C39 to C24, C40 to C25, C41 to C26, C42 to C27, C43 to C28, C44 to C29, C45 to C30, C46 to C31, C47 to C32, C48 to C33, C49 to C34, C50 to C35, D115 to D100, D116 to D101, D117 to D102, D118 to D103, D119 to D104, D120 to D105, D121 to D106, D122 to D107, D109 to D94, D110 to D95, D111 to D96, D112 to D97, D113 to D98, D114 to D99
Connections:
- net LED_OUT: now also D107.2 (DOUT)

Commit message: Update to new keyboard layout
Parts:
- renumbered C22 to C143, C23 to C144, C24 to C145, C25 to C146, C26 to C147, C27 to C148, C28 to C149, C29 to C150, C30 to C151, C31 to C152, C32 to C153, C33 to C154, C34 to C155, C35 to C156, D94 to D143, D95 to D144, D96 to D145, D97 to D146, D98 to D147, D99 to D148, D100 to D149, D101 to D150, D102 to D151, D103 to D152, D104 to D153, D105 to D154, D106 to D155, D107 to D156

Commit message: Convert to kicad 6.0
Parts:
- renumbered C143 to C129, C144 to C130, C145 to C131, C146 to C132, C147 to C133, C148 to C134, C149 to C135, C150 to C136, C151 to C137, C152 to C138, C153 to C139, C154 to C140, C155 to C141, C156 to C142, D143 to D129, D144 to D130, D145 to D131, D146 to D132, D147 to D133, D148 to D134, D149 to D135, D150 to D136, D151 to D137, D152 to D138, D153 to D139, D154 to D140, D155 to D141, D156 to D142

Commit message: Switch to nRF58420 module and battery power
Parts:
- renumbered C129 to C73, C130 to C74, C131 to C75, C132 to C76, C133 to C77, C134 to C78, C135 to C79, C136 to C80, C137 to C81, C138 to C82, C139 to C83, C140 to C84, C141 to C85, C142 to C86, D129 to D149, D130 to D150, D131 to D151, D132 to D152, D133 to D153, D134 to D154, D135 to D155, D136 to D156, D137 to D157, D138 to D158, D139 to D159, D140 to D160, D141 to D161, D142 to D162
