File: main/led_row_14.kicad_sch (KiCad schematic)
At the start: 28 parts

Commit message: routing work
Parts:
- renumbered C73 to C59, C74 to C60, C75 to C61, C76 to C62, C77 to C63, C78 to C64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
